File: Hardware/PCB/clock/clock.kicad_sch (KiCad schematic)
At the start: 12 parts, among them J1 Synth_power_2x5

Commit message: Initial schematic and software
Parts:
- removed C2: 10uF, ao_tht:CP_Radial_D6.3mm_P2.50mm, symbol Device:CP
- removed C4: 100nF, ao_tht:C_Disc_D3.0mm_W1.6mm_P2.50mm, symbol Device:C
- removed D2: 1N5817, ao_tht:D_DO-41_SOD81_P10.16mm_Horizontal, symbol Device:D_Schottky
- removed TP?: -12V, ao_tht:TestPoint_THTPad_D1.5mm_Drill0.7mm, symbol ao_symbols:TestPoint
- added C2, C4, C5, C6: 100nF, ao_tht:C_Disc_D3.0mm_W1.6mm_P2.50mm, symbol ao_symbols:C
- added D2: 1N4148, ao_tht:D_DO-35_SOD27_P7.62mm_Horizontal, symbol ao_symbols:1N4148
- added D3, D4, D5, D6, D7: LED_green, symbol ao_symbols:LED_green
- added J2, J3, J4, J5, J6, J7: AudioJack2, ao_tht:Jack_6.35mm_PJ_629HAN_slots, symbol ao_symbols:AudioJack2
- added OLED1: OLED_128X64, symbol ao_symbols:OLED_128X64_G_V
- added Q1: 2N3904, ao_tht:TO-92_Inline_Wide, symbol ao_symbols:2N3904
- added R1: 100k, ao_tht:R_Axial_DIN0207_L6.3mm_D2.5mm_P10.16mm_Horizontal, symbol ao_symbols:R
- added R10, R11, R2, R3, R4, R5, R7, R8, R9: 10k, ao_tht:R_Axial_DIN0207_L6.3mm_D2.5mm_P10.16mm_Horizontal, symbol ao_symbols:R
- added R12, R13, R14, R15, R16: RL, ao_tht:R_Axial_DIN0207_L6.3mm_D2.5mm_P10.16mm_Horizontal, symbol ao_symbols:R
- added R17, R18, R19, R20, R21: 1k, ao_tht:R_Axial_DIN0207_L6.3mm_D2.5mm_P10.16mm_Horizontal, symbol ao_symbols:R
- added R6: 1M, ao_tht:R_Axial_DIN0207_L6.3mm_D2.5mm_P10.16mm_Horizontal, symbol ao_symbols:R
- added SW1: RotaryEncoder, symbol Device:RotaryEncoder_Switch
- added SW2: SW_Push, symbol ao_symbols:SW_Push
- added TP3: +5V, ao_tht:TestPoint_THTPad_D1.5mm_Drill0.7mm, symbol ao_symbols:TestPoint
- added U1: 40106, symbol 4xxx:40106
- A1: footprint ao_tht:Arduino_Nano -> Module:Arduino_Nano; symbol MCU_Module:Arduino_Nano_v3.x -> ao_symbols:Arduino_Nano_v3.x; SKU (none) -> A-2864; Vendor (none) -> Tayda
- C1: symbol Device:CP -> ao_symbols:CP
- C3: symbol Device:C -> ao_symbols:C
- D1: symbol Device:D_Schottky -> ao_symbols:1N5817
- TP1: renamed from TP?; Config (none) -> DNF
- TP2: renamed from TP?; footprint ao_tht:TestPoint_THTPad_1.5x1.5mm_Drill0.7mm -> ao_tht:TestPoint_THTPad_D1.5mm_Drill0.7mm; Config (none) -> DNF
Connections:
- net +12V: now also A1.30 (VIN)
- net GND: now also A1.29 (GND), A1.4 (GND), C2.2, C4.2, C5.2, C6.2, D2.2 (A), D3.1 (K), D4.1 (K), D5.1 (K), D6.1 (K), D7.1 (K), J2.S, J3.S, J4.S, J5.S, J6.S, J7.S, OLED1.1 (GND), Q1.1 (E), R6.2, SW1.C, SW1.S2, SW2.1, U1.11, U1.13, U1.7 (VSS)
- net ENC_A: now reaches A1.10 (D7)
- net ENC_A: now also U1.2
- net ENC_B: now reaches A1.11 (D8)
- net ENC_B: now also U1.4
- net ENC_PUSH: now reaches A1.12 (D9)
- net ENC_PUSH: now also U1.6
- net TACT: now reaches A1.13 (D10)
- net TACT: now also U1.8
- net CLOCK_IN: now reaches A1.14 (D11)
- net CLOCK_IN: now also Q1.3 (C), R11.2
- net SCA: now reaches A1.23 (A4)
- net SCA: now also OLED1.4 (SDA)
- net SCL: now reaches A1.24 (A5)
- net SCL: now also OLED1.3 (SCL)
- net +5V: now reaches A1.27 (+5V)
- net +5V: now also OLED1.2 (VCC), R11.1, R2.1, R3.1, R4.1, R5.1, TP3.1, U1.14 (VDD)
- net CLOCK_OUT: now reaches A1.5 (D2)
- net CLOCK_OUT: now also R12.2, R17.1
- net DIV_2: now reaches A1.6 (D3)
- net DIV_2: now also R13.2, R18.1
- net DIV_4: now reaches A1.7 (D4)
- net DIV_4: now also R14.2, R19.1
- net DIV_8: now reaches A1.8 (D5)
- net DIV_8: now also R15.2, R20.1
- net DIV_N: now reaches A1.9 (D6)
- net DIV_N: now also R16.2, R21.1
- net -12_IN: no longer names the net of J1.1 (-12V), J1.2 (-12V)
- new net: R2.2, R7.1, SW1.A
- new net: C2.1, R7.2, U1.1
- new net: R10.1, R5.2, SW2.2
- new net: R4.2, R9.1, SW1.S1
- new net: C6.1, R10.2, U1.9
- new net: C4.1, R8.2, U1.3
- new net: D2.1 (K), Q1.2 (B), R1.1, R6.1
- new net: D3.2 (A), R12.1
- new net: D4.2 (A), R13.1
- new net: D6.2 (A), R15.1
- new net: C5.1, R9.2, U1.5
- new net: D5.2 (A), R14.1
- new net: D7.2 (A), R16.1
- new net: R3.2, R8.1, SW1.B
- new net CLK_IN_J: J2.T, R1.2
- new net CLK_OUT_J: J3.T, R17.2
- new net DIV_2_J: J4.T, R18.2
- new net DIV_4_J: J5.T, R19.2
- new net DIV_8_J: J6.T, R20.2
- new net DIV_N_J: J7.T, R21.2
- no-connect marks 0 -> 16
Other:
- title: (none) -> Clock
- moved on the sheet: A1, GRAF1
