File: Hardware/PCB/clock/clock.kicad_pcb (KiCad board)
At the start: 2 copper layers, 146 x 170.5 mm, 67 parts, among them J1 Conn_02x04_Odd_Even, J2 Synth_power_2x5, J3 Conn_02x04_Odd_Even, J4 AudioJack2, J5 AudioJack2, J6 AudioJack2, J7 AudioJack2, J8 AudioJack2, J9 AudioJack2, SW1 SW_Push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

Commit message: Add version # to PCBs; update errata section in build.md
Other:
- board text added: "CLOCK v1.0 Controls board"
- board text added: "CLOCK v1.0 Rich Holmes 11/2022 CC0 1.0"
- board text removed: "CLOCK Controls board"
- board text removed: "CLOCK Rich Holmes 7/2022 CC0 1.0"
Changed lines of the file:
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@@
     (effects (font (size 1 1) (thickness 0.15)) (justify mirror))
   )
-  (gr_text "CLOCK\nRich Holmes\n7/2022 CC0 1.0" (at 70.495 78.74) (layer "B.SilkS")
+  (gr_text "CLOCK v1.0\nRich Holmes\n11/2022 CC0 1.0" (at 70.495 78.74) (layer "B.SilkS")
     (effects (font (size 1 1) (thickness 0.15)) (justify mirror))
   )
@@
     (effects (font (size 1 1) (thickness 0.15)) (justify mirror))
   )
-  (gr_text "CLOCK\nControls board" (at 179.715 85.09) (layer "B.SilkS")
+  (gr_text "CLOCK v1.0\nControls board" (at 179.715 85.09) (layer "B.SilkS")
     (effects (font (size 1 1) (thickness 0.15)) (justify mirror))
   )
