File: Hardware/Panel/clock_panel/clock_panel.kicad_sch (KiCad schematic)
At the start: 18 parts

Commit message: typo; OLED panel footprint
Parts:
- added OLED1: OLED_128X64_Hole, Kosmo_panel:OLED_128x64_1.3in, symbol Kosmo:OLED_128X64_Hole
Changed lines of the file:
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@@
     (pin "1")
+  )
+  (symbol (lib_id "Kosmo:OLED_128X64_Hole") (at 148.59 96.52 0) (unit 1)
+    (in_bom yes) (on_board yes) (fields_autoplaced)
+    (property "Reference" "OLED1" (id 0) (at 155.575 95.6853 0)
+      (effects (font (size 1.27 1.27)) (justify left))
+    )
+    (property "Value" "OLED_128X64_Hole" (id 1) (at 155.575 98.2222 0)
+      (effects (font (size 1.27 1.27)) (justify left))
+    )
+    (property "Footprint" "Kosmo_panel:OLED_128x64_1.3in" (id 2) (at 148.59 96.52 0)
+      (effects (font (size 1.27 1.27)) hide)
+    )
+    (property "Datasheet" "" (id 3) (at 148.59 96.52 0)
+      (effects (font (size 1.27 1.27)) hide)
+    )
   )
   (symbol (lib_id "Kosmo:Led_Hole") (at 114.3 50.8 0) (unit 1)
@@
       (reference "H15") (unit 1) (value "Led_Hole") (footprint "Kosmo_panel:Kosmo_LED_Hole")
     )
-  )
+    (path "/22966d43-d50c-4ced-b35e-ff0ff094ade9"
+      (reference "OLED1") (unit 1) (value "OLED_128X64_Hole") (footprint "Kosmo_panel:OLED_128x64_1.3in")
+    )
+  )
