File: Hardware/PCB/clock/Separate_PCBs/clock_b1.kicad_pcb (KiCad board)
At the start: 2 copper layers, 46 x 142.5 mm, 44 parts, among them J2 Synth_power_2x5, J3 Conn_02x04_Odd_Even, J4 AudioJack2, J5 AudioJack2, J6 AudioJack2, J7 AudioJack2, J8 AudioJack2, J9 AudioJack2, U1 40106

Commit message: new Gerbers
Other:
- board text added: "CLOCK v1.0 Rich Holmes 11/2022 CC0 1.0"
- board text added: "Green"
- board text added: "Red"
- board text removed: "CLOCK Rich Holmes 7/2022 CC0 1.0"
