File: Hardware/PCB/clock/Separate_PCBs/clock_b2.kicad_pcb (KiCad board)
At the start: 2 copper layers, 46 x 93 mm, 20 parts, among them J1 Conn_02x04_Odd_Even, SW1 SW_Push, SW2 RotaryEncoder

Commit message: new Gerbers
Parts:
- turned SW1 to 180 degrees
Routing:
- net Board_0-Net-(R1-Pad2): track 9.74 -> 22.2 mm
Other:
- board text added: "CLOCK v1.0 Controls board"
- board text removed: "CLOCK Controls board"
